File: pcb/Bottom_Plate.kicad_pcb (KiCad board)
At the start: 2 copper layers, 140 x 91.2 mm, 5 parts

Commit message: WIP
Parts:
- removed ? (x3): , 
- removed the REF** at (95.9, 12.6)
- added REF**: MountingHole_2.2mm_M2_Pad_Via, MountingHole:MountingHole_2.2mm_M2_Pad_Via, F.Cu at (275.7, 174.1)
- added REF**: MountingHole_2.2mm_M2_Pad_Via, MountingHole:MountingHole_2.2mm_M2_Pad_Via, F.Cu at (270.9, 134.5)
- added REF**: MountingHole_2.2mm_M2_Pad_Via, MountingHole:MountingHole_2.2mm_M2_Pad_Via, F.Cu at (149.7, 169.8)
- added REF**: MountingHole_2.2mm_M2_Pad_Via, MountingHole:MountingHole_2.2mm_M2_Pad_Via, F.Cu at (214.8, 185.0)
- added REF**: MountingHole_2.2mm_M2_Pad_Via, MountingHole:MountingHole_2.2mm_M2_Pad_Via, F.Cu at (153.8, 134.2)
- added REF**: MountingHole_2.2mm_M2_Pad_Via, MountingHole:MountingHole_2.2mm_M2_Pad_Via, F.Cu at (215.3, 115.7)
- added Ref**: Val**, kiboard_cache:backleft-svg2shenzen, F.Cu at (214.3, 158.1)
- added Ref**: Val**, kiboard_cache:backright-copper, F.Cu at (213.6, 157.0)
- moved REF** 232.6 mm to (204.2, 143.2)
