File: pcb/Wubbo.kicad_pcb (KiCad board)
At the start: 2 copper layers, 140 x 91.2 mm, 50 parts, among them J1 USB_C_Receptacle, J2 SWD, J3 USB, Q1 AO3407, Q2 AO3407, SW1 Choc, SW10 Choc, SW11 Choc, SW12 Choc, SW13 Choc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

Commit message: WIP
Parts:
- added J3: USB, Connector_PinSocket_1.00mm:PinSocket_1x04_P1.00mm_Vertical, F.Cu at (122.0, -32.0)
- added Ref**: Val**, kiboard_cache:frontleft-2, F.Cu at (59.4, -12.7)
- added Ref**: Val**, kiboard_cache:frontright-1, F.Cu at (53.5, -10.9)
- added Ref**: Val**, kiboard_cache:frontright-2, F.Cu at (-38.0, -11.7)
- added Ref**: Val**, kiboard_cache:frontleft-1, F.Cu at (58.3, -11.2)
- ? (x3): value (none) -> MountingHole_2.2mm_M2_Pad_Via; footprint (none) -> MountingHole:MountingHole_2.2mm_M2_Pad_Via
- SW1, SW10, SW11, SW12, SW13, SW14, SW15, SW16, SW17, SW2, SW3, SW4, SW5, SW6, SW7, SW8, SW9: footprint kicad-keyboard-parts:PG13500-reversible -> kiboard_cache:PG13500-reversible
- moved SW10 0.40 mm to (92.7, -21.5)
- moved SW15 0.40 mm to (92.1, -4.56)
- moved SW5 0.40 mm to (93.3, -38.5)
- moved SW14 0.20 mm to (74.0, -9.87)
- moved SW9 0.20 mm to (74.3, -26.9)
- moved SW4 0.20 mm to (74.6, -43.9)
Connections:
- BAT pad 2: -BATT -> GND
- U1 pad 6: unconnected-(U1-Pad6) -> P0.03
- U1 pad 7: unconnected-(U1-Pad7) -> P0.02
Routing:
- net P0.02: track 0.00 -> 15.7 mm
- net P0.03: track 0.00 -> 14.1 mm
- net EXT_VCC: track 1.04 -> 13.7 mm, vias 1 -> 0
- net SW16: track 63.2 -> 61.9 mm
Other:
- board text added: "P0.02"
- board text added: "P0.03"
- board text added: "VCC"
