File: KiCad/Wubbo.kicad_pcb (KiCad board)
At the start: 2 copper layers, 140 x 91.2 mm, 55 parts, among them J1 USB_C_Receptacle, J2 SWD, J3 USB, Q1 AO3407, Q2 AO3407, SW1 Choc, SW10 Choc, SW11 Choc, SW12 Choc, SW13 Choc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

Commit message: wip
Parts:
- U2: value XC6206P -> XC6206P LDO
- U3: value LTC4054 -> LTC4054ES5-4.2
- renumbered BAT to J4, R_TACT2 to R_TACT1
Connections:
- J1 pad 10: (no net) -> /Net-(J1-CC1)
- J1 pad 13: GND -> (no net)
- J1 pad 5: USBD+ -> USBD-
- J1 pad 6: USBD- -> USBD+
- J1 pad 7: USBD+ -> USBD-
- J1 pad 8: USBD- -> USBD+
- J1 pad 9: /Net-(J1-CC1) -> (no net)
- J4 pad 2: GND -> -BATT
- U1 pad 6: P0.03 -> unconnected-(U1-Pad6)
- U1 pad 7: P0.02 -> unconnected-(U1-Pad7)
Routing:
- net unconnected-(U1-Pad7): track 0.00 -> 15.7 mm
- net P0.02: track 15.7 -> 0.00 mm
- net unconnected-(U1-Pad6): track 0.00 -> 14.1 mm
- net P0.03: track 14.1 -> 0.00 mm
- net USBD-: track 11.3 -> 10.6 mm, vias 3 -> 0
- net USBD+: track 11.3 -> 11.5 mm, vias 0 -> 2

Commit message: WIP
Parts:
- J4: moved to F.Cu
- moved R8 3.65 mm to (117.6, -26.8), turned to 90 degrees
- moved J4 1.56 mm to (120.5, -23.0), turned to 180 degrees
- moved D2 0.41 mm to (115.9, -28.5)
- moved R7 0.39 mm to (116.0, -25.3)
- moved U3 0.22 mm to (120.2, -26.5), turned to 90 degrees
Connections:
- D2 pad 2: CHRG_LED -> VBUS
- J4 pad 2: -BATT -> GND
- R7 pad 2: GND -> Net-(U3-Pad1)
- U3 pad 1: CHRG_LED -> Net-(U3-Pad1)
Routing:
- net unconnected-(U1-Pad7): track 15.7 -> 0.00 mm
- net P0.02: track 0.00 -> 15.7 mm
- net unconnected-(U1-Pad6): track 14.1 -> 0.00 mm
- net P0.03: track 0.00 -> 14.1 mm
- net VBUS: track 82.7 -> 88.9 mm
- net CHRG_LED: track 3.27 -> 0.00 mm
- net Net-(U3-Pad1): track 0.00 -> 3.08 mm
- net GND: track 18.9 -> 16.5 mm
- net +BATT: track 19.1 -> 18.2 mm

Commit message: WIP
Parts:
- J2, J3: footprint Connector_PinSocket_1.00mm:PinSocket_1x04_P1.00mm_Vertical -> Connector_PinSocket_2.00mm:PinSocket_1x04_P2.00mm_Vertical
- J5: renamed from J3; footprint Connector_PinSocket_1.00mm:PinSocket_1x04_P1.00mm_Vertical -> Connector_PinHeader_2.00mm:PinHeader_1x04_P2.00mm_Vertical
- moved J3 4.00 mm to (115.1, -14.1), turned to 0 degrees
- moved J2 3.87 mm to (118.1, -14.2), turned to 0 degrees
- moved J5 2.08 mm to (122.6, -30.0), turned to 11 degrees
Connections:
- J1 pad 13: (no net) -> GND
- J2 pad 3: SWDIO -> SWDCLK
- J2 pad 4: SWDCLK -> SWDIO
- U1 pad 6: unconnected-(U1-Pad6) -> P0.03
- U1 pad 7: unconnected-(U1-Pad7) -> P0.02
Routing:
- net +3V3: track 29.0 -> 22.3 mm
- net P0.03: track 14.1 -> 8.81 mm
- net VBUS: track 88.9 -> 83.9 mm
- net P0.02: track 15.7 -> 10.9 mm
- net D-: track 40.8 -> 36.9 mm
- net D+: track 40.1 -> 37.0 mm
- net SWDIO: track 5.32 -> 2.93 mm
- net GND: track 16.5 -> 15.0 mm
- net EXT_VCC: track 13.7 -> 12.4 mm
