File: KiCad/Wubbo.kicad_pcb (KiCad board)
At the start: 2 copper layers, 140 x 91.2 mm, 55 parts, among them J1 USB_C_Receptacle, J2 SWD, J3 USB, J4 JST-BATT, J5 USB, Q1 AO3407, Q2 AO3407, SW1 Choc, SW10 Choc, SW11 Choc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

Commit message: WIP
Parts:
- ? (x3), REF**: footprint MountingHole:MountingHole_2.2mm_M2_Pad_Via -> kiboard_cache:MountingHole_2.2mm_M2_Pad_Via

Commit message: wip
Parts:
- added C3: 4.7n, Capacitor_SMD:C_0603_1608Metric, F.Cu at (112.8, -40.0)
- added R10: 1M, Resistor_SMD:R_0603_1608Metric, F.Cu at (110.7, -39.9)
- moved J4 42.0 mm to (88.8, 4.56), turned to -90 degrees
Connections:
- R1 pad 1: /Net-(J1-CC2) -> Net-(R1-Pad1)
- R2 pad 1: /Net-(J1-CC1) -> Net-(J1-PadB5)
Routing:
- net +BATT: track 18.2 -> 12.7 mm
- net Earth: track 0.00 -> 4.72 mm
- net Net-(J1-PadB5): track 0.00 -> 3.40 mm
- net /Net-(J1-CC1): track 3.40 -> 0.00 mm
- net Net-(R1-Pad1): track 0.00 -> 2.73 mm
- net /Net-(J1-CC2): track 2.73 -> 0.00 mm

Commit message: wip
Parts:
- moved J4 0.38 mm to (89.2, 4.72)
Routing:
- net +BATT: track 12.7 -> 78.7 mm, vias 1 -> 5
Changed lines of the file:
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@@
   )
   (footprint "Connector_JST:JST_PH_S2B-PH-K_1x02_P2.00mm_Horizontal" (layer "F.Cu")
-    (at 88.82 4.56 -90)
+    (at 89.17 4.72 -90)
     (descr "JST PH series connector, S2B-PH-K (http://www.jst-mfg.com/product/pdf/eng/ePH.pdf), generated with kicad-footprint-generator")
     (tags "connector JST PH top entry")
@@
     )
   )
-  (gr_arc (start 102.69 -6.97) (mid 98.480436 1.844721) (end 89.1 4.57) (layer "F.Cu") (width 0.2))
-  (gr_line (start 102.69 -6.97) (end 102.69 -34.78) (layer "F.Cu") (width 0.2))
-  (gr_arc (start 102.68 -32.19) (mid 107.03974 -35.811495) (end 112.57 -34.64) (layer "B.Cu") (width 0.2))
   (gr_rect (start 111.14 -21.975) (end 114.27 -20.365) (layer "Cmts.User") (width 0.1) (fill solid))
   (gr_rect (start 104.5 -21.705) (end 107.63 -20.095) (layer "Cmts.User") (width 0.1) (fill solid))
@@
   (segment (start 110.003372 -18.721818) (end 110 -21) (width 0.25) (layer "F.Cu") (net 6))
   (segment (start 110.025 -21.15) (end 111.8 -21.15) (width 0.2) (layer "F.Cu") (net 6))
-  (segment (start 116.575 -36.575) (end 117.471204 -37.312719) (width 0.25) (layer "F.Cu") (net 7))
-  (segment (start 116.5 -35.9) (end 116.575 -36.575) (width 0.25) (layer "F.Cu") (net 7))
+  (segment (start 102.69 -6.97) (end 102.69 -31.23) (width 0.3) (layer "F.Cu") (net 7))
+  (segment (start 121.19 -24.44) (end 121.17 -25.4025) (width 0.3) (layer "F.Cu") (net 7))
+  (via (at 121.19 -24.44) (size 0.4) (drill 0.2) (layers "F.Cu" "B.Cu") (free) (net 7))
+  (via (at 116.475 -31.815) (size 0.4) (drill 0.2) (layers "F.Cu" "B.Cu") (net 7))
   (via (at 116.5 -35.9) (size 0.8) (drill 0.4) (layers "F.Cu" "B.Cu") (net 7))
-  (segment (start 116.5 -35.9) (end 116.475 -35.399692) (width 0.25) (layer "B.Cu") (net 7))
-  (segment (start 117.35368 -27.79632) (end 118.071321 -27.078679) (width 0.25) (layer "B.Cu") (net 7))
-  (segment (start 116.475 -35.399692) (end 116.475 -29.917641) (width 0.25) (layer "B.Cu") (net 7))
-  (segment (start 116.5 -35.9) (end 116.987657 -35.912349) (width 0.2) (layer "B.Cu") (net 7))
-  (segment (start 116.987657 -35.912349) (end 118.008756 -35.912349) (width 0.2) (layer "B.Cu") (net 7))
-  (arc (start 117.35368 -27.79632) (mid 116.703361 -28.76959) (end 116.475 -29.917641) (width 0.25) (layer "B.Cu") (net 7))
+  (via (at 103.19 -32.53) (size 0.4) (drill 0.2) (layers "F.Cu" "B.Cu") (net 7))
+  (via (at 113.16 -35.12) (size 0.4) (drill 0.2) (layers "F.Cu" "B.Cu") (net 7))
+  (arc (start 113.13 -35.14) (mid 115.18037 -33.883514) (end 116.46 -31.85) (width 0.3) (layer "F.Cu") (net 7))
+  (arc (start 116.5 -35.89) (mid 116.693766 -36.71453) (end 117.35 -37.25) (width 0.3) (layer "F.Cu") (net 7))
+  (arc (start 102.69 -31.23) (mid 102.802317 -31.930011) (end 103.18 -32.53) (width 0.3) (layer "F.Cu") (net 7))
+  (arc (start 102.69 -6.97) (mid 98.480436 1.844721) (end 89.1 4.57) (width 0.3) (layer "F.Cu") (net 7))
+  (segment (start 116.5 -35.9) (end 116.475 -35.399692) (width 0.3) (layer "B.Cu") (net 7))
+  (segment (start 116.475 -31.815) (end 116.475 -29.917641) (width 0.3) (layer "B.Cu") (net 7))
+  (segment (start 116.475 -35.399692) (end 116.475 -31.815) (width 0.3) (layer "B.Cu") (net 7))
+  (segment (start 116.5 -35.9) (end 116.987657 -35.912349) (width 0.3) (layer "B.Cu") (net 7))
+  (segment (start 116.987657 -35.912349) (end 118.008756 -35.912349) (width 0.3) (layer "B.Cu") (net 7))
+  (arc (start 121.2 -24.44) (mid 117.855644 -26.354283) (end 116.47 -29.95) (width 0.3) (layer "B.Cu") (net 7))
+  (arc (start 103.16 -32.5) (mid 107.745625 -35.390569) (end 113.16 -35.13) (width 0.3) (layer "B.Cu") (net 7))
   (segment (start 107.403372 -9.771818) (end 108.040227 -9.960151) (width 0.25) (layer "F.Cu") (net 8))
   (segment (start 113.070238 -13.374805) (end 113.51 -13.935) (width 0.25) (layer "F.Cu") (net 8))
