File: KiCad/Wubbo.kicad_pcb (KiCad board)
At the start: 2 copper layers, 140 x 91.2 mm, 57 parts, among them J1 USB_C_Receptacle, J2 SWD, J3 USB, J4 JST-BATT, J5 USB, Q1 AO3407, Q2 AO3407, SW1 Choc, SW10 Choc, SW11 Choc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

Commit message: wip
Parts:
- removed the R_TACT1 at (98.2, -51.3) (x2)
- added ?: , clipboard:9b7f651c-c6a4-4f53-b457-ec411c8fc700, F.Cu at (-4.69, -5.51)
- added ?: , clipboard:9b7f651c-c6a4-4f53-b457-ec411c8fc700, B.Cu at (5.67, -6.35)
- added R_TACT1: SW_Push, kiboard_cache:3-4-2_micro_tact_switch, F.Cu at (115.6, -45.1)
- C3: footprint Capacitor_SMD:C_0603_1608Metric -> Capacitor_SMD:C_0805_2012Metric
- D1: footprint LED_SMD:LED_0603_1608Metric -> kiboard_cache:LED_0603_1608Metric_shinethrough
- moved C3 15.8 mm to (100.1, -49.5), turned to -15.5 degrees
- moved R10 13.3 mm to (99.5, -47.2), turned to -15.5 degrees
- moved J4 10.5 mm to (79.1, 7.59)
- moved D2 1.44 mm to (116.0, -27.0)
- moved D1 1.40 mm to (114.1, -27.1)
- moved R7 1.28 mm to (116.0, -24.1)
- moved R6 1.18 mm to (114.1, -24.1)
Routing:
- net RESET: track 62.8 -> 35.9 mm, vias 2 -> 1
- net +BATT: track 78.8 -> 89.1 mm
- net BLUE_LED: track 17.3 -> 16.0 mm, vias 2 -> 1
- net Earth: track 4.72 -> 5.67 mm
- net /BAT+_SWITCHED: track 28.4 -> 27.5 mm
- net Net-(R7-Pad2): track 3.08 -> 3.92 mm

Commit message: wip
Parts:
- GR3, GR4, GR5, GR6: renamed from Ref**; value Val** -> (none)
- gave numbers to parts that had none: 2
- renumbered REF** to TENT1
Changed lines of the file:
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@@
   (title_block
     (title "Wubbo")
-    (rev "v0.1")
+    (rev "v0.2")
     (company "cache.works")
   )
@@
   (footprint "clipboard:9b7f651c-c6a4-4f53-b457-ec411c8fc700" (layer "F.Cu")
     (at -4.691213 -5.507578 5)
-    (fp_text reference "" (at 0 0 5) (layer "F.SilkS")
+    (fp_text reference "GR1" (at 0 0 5) (layer "F.SilkS")
       (effects (font (size 1.27 1.27) (thickness 0.15)))
     )
@@
     (at 59.445876 -12.66613)
     (attr through_hole)
-    (fp_text reference "Ref**" (at 0 0) (layer "F.SilkS") hide
+    (fp_text reference "GR4" (at 0 0) (layer "F.SilkS") hide
       (effects (font (size 1.27 1.27) (thickness 0.15)))
     )
-    (fp_text value "Val**" (at 0 0) (layer "F.SilkS") hide
+    (fp_text value "" (at 0 0) (layer "F.SilkS") hide
       (effects (font (size 1.27 1.27) (thickness 0.15)))
     )
@@
     (at 53.48 -10.865)
     (attr through_hole)
-    (fp_text reference "Ref**" (at 0 0) (layer "F.SilkS") hide
+    (fp_text reference "GR5" (at 0 0) (layer "F.SilkS") hide
       (effects (font (size 1.27 1.27) (thickness 0.15)))
     )
-    (fp_text value "Val**" (at 0 0) (layer "F.SilkS") hide
+    (fp_text value "" (at 0 0) (layer "F.SilkS") hide
       (effects (font (size 1.27 1.27) (thickness 0.15)))
     )
@@
     (property "Sheetname" "")
     (attr smd)
-    (fp_text reference "R4" (at 0.005 1.335 180) (layer "F.SilkS")
+    (fp_text reference "R4" (at 1.725 0.035 180) (layer "F.SilkS")
       (effects (font (size 0.6 0.6) (thickness 0.1)))
     )
@@
     (at -38.049357 -11.67519)
     (attr through_hole)
-    (fp_text reference "Ref**" (at 0 0) (layer "F.SilkS") hide
+    (fp_text reference "GR3" (at 0 0) (layer "F.SilkS") hide
       (effects (font (size 1.27 1.27) (thickness 0.15)))
     )
-    (fp_text value "Val**" (at 0 0) (layer "F.SilkS") hide
+    (fp_text value "" (at 0 0) (layer "F.SilkS") hide
       (effects (font (size 1.27 1.27) (thickness 0.15)))
     )
@@
     (tags "mounting hole 2.2mm m2")
     (attr exclude_from_pos_files exclude_from_bom)
-    (fp_text reference "REF**" (at 0 -3.2) (layer "F.SilkS")
+    (fp_text reference "REF**" (at 0 -3.2) (layer "F.SilkS") hide
       (effects (font (size 1 1) (thickness 0.15)))
     )
@@
     (property "Sheetname" "")
     (attr smd)
-    (fp_text reference "R5" (at 0.005 -1.085) (layer "F.SilkS")
+    (fp_text reference "R5" (at -0.015 1.05) (layer "F.SilkS")
       (effects (font (size 0.6 0.6) (thickness 0.1)))
     )
@@
       (effects (font (size 1 1) (thickness 0.15)))
     )
-    (fp_line (start -1.4 1.73) (end -1.4 3.02) (layer "F.SilkS") (width 0.12))
-    (fp_line (start -3.45 -0.07) (end -3.45 0.72) (layer "F.SilkS") (width 0.12))
-    (fp_line (start -2.85 1.73) (end 2.85 1.73) (layer "F.SilkS") (width 0.12))
-    (fp_line (start -1.4 3.02) (end -1.2 3.23) (layer "F.SilkS") (width 0.12))
-    (fp_line (start -1.2 3.23) (end -0.3 3.23) (layer "F.SilkS") (width 0.12))
-    (fp_line (start 1.4 -1.12) (end 1.6 -1.12) (layer "F.SilkS") (width 0.12))
-    (fp_line (start 3.45 0.72) (end 3.45 -0.07) (layer "F.SilkS") (width 0.12))
-    (fp_line (start -0.1 3.02) (end -0.3 3.23) (layer "F.SilkS") (width 0.12))
-    (fp_line (start -0.1 3.02) (end -0.1 1.73) (layer "F.SilkS") (width 0.12))
-    (fp_line (start -1.6 -1.12) (end 0.1 -1.12) (layer "F.SilkS") (width 0.12))
     (fp_line (start 1.65 3.4) (end -1.65 3.4) (layer "F.CrtYd") (width 0.05))
     (fp_line (start 4.4 2.1) (end 1.65 2.1) (layer "F.CrtYd") (width 0.05))
@@
     (at 58.31 -11.195)
     (attr through_hole)
-    (fp_text reference "Ref**" (at 0 0) (layer "F.SilkS") hide
+    (fp_text reference "GR6" (at 0 0) (layer "F.SilkS") hide
       (effects (font (size 1.27 1.27) (thickness 0.15)))
     )
-    (fp_text value "Val**" (at 0 0) (layer "F.SilkS") hide
+    (fp_text value "" (at 0 0) (layer "F.SilkS") hide
       (effects (font (size 1.27 1.27) (thickness 0.15)))
     )
@@
       (effects (font (size 1 1) (thickness 0.15)))
     )
-    (fp_line (start -1.06 1) (end -1.06 7.06) (layer "F.SilkS") (width 0.12))
-    (fp_line (start 1.06 1) (end 1.06 7.06) (layer "F.SilkS") (width 0.12))
-    (fp_line (start -1.06 -1.06) (end 0 -1.06) (layer "F.SilkS") (width 0.12))
-    (fp_line (start -1.06 1) (end 1.06 1) (layer "F.SilkS") (width 0.12))
-    (fp_line (start -1.06 7.06) (end 1.06 7.06) (layer "F.SilkS") (width 0.12))
-    (fp_line (start -1.06 0) (end -1.06 -1.06) (layer "F.SilkS") (width 0.12))
     (fp_line (start 1.5 7.5) (end 1.5 -1.5) (layer "F.CrtYd") (width 0.05))
     (fp_line (start -1.5 -1.5) (end -1.5 7.5) (layer "F.CrtYd") (width 0.05))
@@
     (tags "splitkb tenting puck")
     (attr through_hole)
-    (fp_text reference "REF**" (at 7.6835 1.4605 3) (layer "F.Fab")
+    (fp_text reference "TENT1" (at 7.6835 1.4605 3) (layer "F.Fab")
       (effects (font (size 1 1) (thickness 0.15)))
     )
@@
   (footprint "clipboard:9b7f651c-c6a4-4f53-b457-ec411c8fc700" (layer "B.Cu")
     (at 5.669519 -6.351834 -175)
-    (fp_text reference "" (at 0 0 5) (layer "B.SilkS")
+    (fp_text reference "GR2" (at 0 0 5) (layer "B.SilkS")
       (effects (font (size 1.27 1.27) (thickness 0.15)) (justify mirror))
     )
@@
       (effects (font (size 1 1) (thickness 0.15)) (justify mirror))
     )
-    (fp_line (start -3.45 0.07) (end -3.45 -0.72) (layer "B.SilkS") (width 0.12))
-    (fp_line (start -2.85 -1.73) (end 2.85 -1.73) (layer "B.SilkS") (width 0.12))
-    (fp_line (start -0.1 -3.02) (end -0.1 -1.73) (layer "B.SilkS") (width 0.12))
-    (fp_line (start -1.4 -1.73) (end -1.4 -3.02) (layer "B.SilkS") (width 0.12))
-    (fp_line (start 1.4 1.12) (end 1.6 1.12) (layer "B.SilkS") (width 0.12))
-    (fp_line (start -1.4 -3.02) (end -1.2 -3.23) (layer "B.SilkS") (width 0.12))
-    (fp_line (start -1.2 -3.23) (end -0.3 -3.23) (layer "B.SilkS") (width 0.12))
-    (fp_line (start -1.6 1.12) (end 0.1 1.12) (layer "B.SilkS") (width 0.12))
-    (fp_line (start 3.45 -0.72) (end 3.45 0.07) (layer "B.SilkS") (width 0.12))
-    (fp_line (start -0.1 -3.02) (end -0.3 -3.23) (layer "B.SilkS") (width 0.12))
     (fp_line (start 1.65 -3.4) (end -1.65 -3.4) (layer "B.CrtYd") (width 0.05))
     (fp_line (start 1.65 -2.1) (end 1.65 -3.4) (layer "B.CrtYd") (width 0.05))
