File: KiCad/Wubbo.kicad_sch (KiCad schematic)
At the start: 44 parts, among them J1 USB_C_Receptacle, J2 SWD, J3 USB, J4 JST-BATT, Q1 AO3407, Q2 AO3407, SW1 Choc, SW10 Choc, SW11 Choc, SW12 Choc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

Commit message: wip
Connections:
- net Net-(J1-CC1): now also J1.10 (CC1); no longer J1.9 (CC1)
- net USBD+: now also J1.6 (D+), J1.8 (D+); no longer J1.5 (D+), J1.7 (D+)
- net USBD-: now also J1.5 (D-), J1.7 (D-); no longer J1.6 (D-), J1.8 (D-)
Changed lines of the file:
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@@
   (junction (at 226.06 165.1) (diameter 0) (color 0 0 0 0)
   )
+  (junction (at 242.57 165.1) (diameter 0) (color 0 0 0 0)
+  )
+  (junction (at 259.08 153.67) (diameter 0) (color 0 0 0 0)
+  )
+  (junction (at 242.57 153.67) (diameter 0) (color 0 0 0 0)
+  )
+  (junction (at 191.77 153.67) (diameter 0) (color 0 0 0 0)
+  )
   (junction (at 130.81 48.26) (diameter 0) (color 0 0 0 0)
-  )
-  (junction (at 242.57 165.1) (diameter 0) (color 0 0 0 0)
-  )
-  (junction (at 259.08 153.67) (diameter 0) (color 0 0 0 0)
-  )
-  (junction (at 242.57 153.67) (diameter 0) (color 0 0 0 0)
-  )
-  (junction (at 191.77 153.67) (diameter 0) (color 0 0 0 0)
   )
   (junction (at 209.55 153.67) (diameter 0) (color 0 0 0 0)
@@
     (stroke (width 0) (type default) (color 0 0 0 0))
   )
+  (wire (pts (xy 130.81 48.26) (xy 130.81 49.53))
+    (stroke (width 0) (type default) (color 0 0 0 0))
+  )
   (wire (pts (xy 209.55 165.1) (xy 209.55 170.18))
     (stroke (width 0) (type default) (color 0 0 0 0))
@@
     (stroke (width 0) (type default) (color 0 0 0 0))
   )
+  (wire (pts (xy 130.81 48.26) (xy 135.89 48.26))
+    (stroke (width 0) (type default) (color 0 0 0 0))
+  )
   (wire (pts (xy 45.72 99.06) (xy 45.72 100.33))
     (stroke (width 0) (type default) (color 0 0 0 0))
@@
     (stroke (width 0) (type default) (color 0 0 0 0))
   )
-  (wire (pts (xy 130.81 53.34) (xy 130.81 52.07))
-    (stroke (width 0) (type default) (color 0 0 0 0))
-  )
-  (wire (pts (xy 130.81 54.61) (xy 130.81 53.34))
-    (stroke (width 0) (type default) (color 0 0 0 0))
-  )
-  (wire (pts (xy 130.81 53.34) (xy 133.35 53.34))
+  (wire (pts (xy 130.81 52.07) (xy 130.81 53.34))
     (stroke (width 0) (type default) (color 0 0 0 0))
   )
@@
     (stroke (width 0) (type default) (color 0 0 0 0))
   )
+  (wire (pts (xy 130.81 53.34) (xy 130.81 54.61))
+    (stroke (width 0) (type default) (color 0 0 0 0))
+  )
   (wire (pts (xy 130.81 41.91) (xy 137.16 41.91))
     (stroke (width 0) (type default) (color 0 0 0 0))
@@
     (stroke (width 0) (type default) (color 0 0 0 0))
   )
-  (wire (pts (xy 130.81 48.26) (xy 133.35 48.26))
-    (stroke (width 0) (type default) (color 0 0 0 0))
-  )
-  (wire (pts (xy 130.81 48.26) (xy 130.81 49.53))
-    (stroke (width 0) (type default) (color 0 0 0 0))
-  )
   (polyline (pts (xy 91.44 118.11) (xy 165.1 118.11))
     (stroke (width 0) (type default) (color 0 0 0 0))
@@
   )
   (polyline (pts (xy 223.52 12.7) (xy 223.52 118.11))
+    (stroke (width 0) (type default) (color 0 0 0 0))
+  )
+  (wire (pts (xy 130.81 53.34) (xy 135.89 53.34))
     (stroke (width 0) (type default) (color 0 0 0 0))
   )
@@
     )
   )
-  (global_label "USBD-" (shape input) (at 133.35 48.26 0) (fields_autoplaced)
-    (effects (font (size 1.27 1.27)) (justify left))
-    (property "Intersheet References" "${INTERSHEET_REFS}" (id 0) (at 142.3266 48.3394 0)
+  (global_label "USBD-" (shape input) (at 135.89 53.34 0) (fields_autoplaced)
+    (effects (font (size 1.27 1.27)) (justify left))
+    (property "Intersheet References" "${INTERSHEET_REFS}" (id 0) (at 144.8666 53.4194 0)
       (effects (font (size 1.27 1.27)) (justify left) hide)
     )
@@
     )
   )
-  (global_label "USBD+" (shape input) (at 133.35 53.34 0) (fields_autoplaced)
-    (effects (font (size 1.27 1.27)) (justify left))
-    (property "Intersheet References" "${INTERSHEET_REFS}" (id 0) (at 142.3266 53.4194 0)
+  (global_label "USBD+" (shape input) (at 135.89 48.26 0) (fields_autoplaced)
+    (effects (font (size 1.27 1.27)) (justify left))
+    (property "Intersheet References" "${INTERSHEET_REFS}" (id 0) (at 144.8666 48.3394 0)
       (effects (font (size 1.27 1.27)) (justify left) hide)
     )
@@
       (effects (font (size 1.27 1.27)) hide)
     )
-    (property "Datasheet" "https://www.usb.org/sites/default/files/documents/usb_type-c.zip" (id 3) (at 130.81 69.85 0)
+    (property "Datasheet" "" (id 3) (at 130.81 69.85 0)
       (effects (font (size 1.27 1.27)) hide)
     )
@@
     (pin "7")
     (pin "8")
-    (pin "9")
+    (pin "10")
     (pin "A1")
     (pin "A12")

Commit message: remove rotary encoder from schematic
Parts:
- removed E1: RotaryEncoder_Switch, rotary_encoder, symbol Device:RotaryEncoder_Switch
Other:
- note removed: "Rotary encoder"
Changed lines of the file:
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@@
-    (stroke (width 0) (type default) (color 0 0 0 0))
-  )
-  (wire (pts (xy 137.16 186.69) (xy 135.89 186.69))
     (stroke (width 0) (type default) (color 0 0 0 0))
   )
@@
   )
   (text "Battery Voltage sensing" (at 176.53 60.96 0)
-    (effects (font (size 2 2)) (justify left bottom))
-  )
-  (text "Rotary encoder" (at 116.84 176.53 0)
     (effects (font (size 2 2)) (justify left bottom))
   )
@@
     )
   )
-  (global_label "ENC1" (shape input) (at 120.65 186.69 180) (fields_autoplaced)
-    (effects (font (size 1.27 1.27)) (justify right))
-    (property "Intersheet References" "${INTERSHEET_REFS}" (id 0) (at 113.3668 186.6106 0)
-      (effects (font (size 1.27 1.27)) (justify right) hide)
-    )
-  )
   (global_label "SW14" (shape input) (at 71.12 66.04 0) (fields_autoplaced)
     (effects (font (size 1.27 1.27)) (justify left))
@@
     )
   )
-  (global_label "ENC2" (shape input) (at 120.65 191.77 180) (fields_autoplaced)
-    (effects (font (size 1.27 1.27)) (justify right))
-    (property "Intersheet References" "${INTERSHEET_REFS}" (id 0) (at 113.3668 191.6906 0)
-      (effects (font (size 1.27 1.27)) (justify right) hide)
-    )
-  )
   (global_label "SW1" (shape input) (at 181.61 142.24 90) (fields_autoplaced)
     (effects (font (size 1.27 1.27)) (justify left))
@@
     (effects (font (size 1.27 1.27)) (justify left))
     (property "Intersheet References" "${INTERSHEET_REFS}" (id 0) (at 215.9 158.0566 90)
-      (effects (font (size 1.27 1.27)) (justify left) hide)
-    )
-  )
-  (global_label "SW18" (shape input) (at 137.16 186.69 0) (fields_autoplaced)
-    (effects (font (size 1.27 1.27)) (justify left))
-    (property "Intersheet References" "${INTERSHEET_REFS}" (id 0) (at 144.5642 186.6106 0)
       (effects (font (size 1.27 1.27)) (justify left) hide)
     )
@@
     (pin "3")
   )
-  (symbol (lib_id "power:GND") (at 120.65 189.23 270) (unit 1)
-    (in_bom yes) (on_board yes) (fields_autoplaced)
-    (property "Reference" "#PWR0114" (id 0) (at 114.3 189.23 0)
-      (effects (font (size 1.27 1.27)) hide)
-    )
-    (property "Value" "GND" (id 1) (at 116.84 189.2299 90)
-      (effects (font (size 1.27 1.27)) (justify right))
-    )
-    (property "Footprint" "" (id 2) (at 120.65 189.23 0)
-      (effects (font (size 1.27 1.27)) hide)
-    )
-    (property "Datasheet" "" (id 3) (at 120.65 189.23 0)
-      (effects (font (size 1.27 1.27)) hide)
-    )
-    (pin "1")
-  )
   (symbol (lib_id "Switch:SW_Push") (at 237.49 153.67 0) (unit 1)
     (in_bom yes) (on_board yes) (fields_autoplaced)
@@
     (pin "1")
     (pin "2")
-  )
-  (symbol (lib_id "power:GND") (at 135.89 191.77 90) (unit 1)
-    (in_bom yes) (on_board yes) (fields_autoplaced)
-    (property "Reference" "#PWR0116" (id 0) (at 142.24 191.77 0)
-      (effects (font (size 1.27 1.27)) hide)
-    )
-    (property "Value" "GND" (id 1) (at 139.7 191.7699 90)
-      (effects (font (size 1.27 1.27)) (justify right))
-    )
-    (property "Footprint" "" (id 2) (at 135.89 191.77 0)
-      (effects (font (size 1.27 1.27)) hide)
-    )
-    (property "Datasheet" "" (id 3) (at 135.89 191.77 0)
-      (effects (font (size 1.27 1.27)) hide)
-    )
-    (pin "1")
   )
   (symbol (lib_id "power:+3.3V") (at 240.03 106.68 90) (unit 1)
@@
     (pin "3")
   )
-  (symbol (lib_id "Device:RotaryEncoder_Switch") (at 128.27 189.23 0) (unit 1)
-    (in_bom yes) (on_board yes) (fields_autoplaced)
-    (property "Reference" "E1" (id 0) (at 128.27 179.07 0))
-    (property "Value" "RotaryEncoder_Switch" (id 1) (at 128.27 181.61 0))
-    (property "Footprint" "rotary_encoder" (id 2) (at 124.46 185.166 0)
-      (effects (font (size 1.27 1.27)) hide)
-    )
-    (property "Datasheet" "~" (id 3) (at 128.27 182.626 0)
-      (effects (font (size 1.27 1.27)) hide)
-    )
-    (pin "A")
-    (pin "B")
-    (pin "C")
-    (pin "S1")
-    (pin "S2")
-  )
   (symbol (lib_id "Switch:SW_Push") (at 220.98 142.24 0) (unit 1)
     (in_bom yes) (on_board yes) (fields_autoplaced)
@@
       (reference "#PWR0113") (unit 1) (value "-BATT") (footprint "")
     )
-    (path "/80ca1a4e-2078-444c-acdb-3aecce2c8de9"
-      (reference "#PWR0114") (unit 1) (value "GND") (footprint "")
-    )
     (path "/3cf0fbfd-66b2-4a7f-b06a-44415f8c69c1"
       (reference "#PWR0115") (unit 1) (value "GND") (footprint "")
     )
-    (path "/83900970-cbf3-4acc-b728-49a88e4fbc21"
-      (reference "#PWR0116") (unit 1) (value "GND") (footprint "")
-    )
     (path "/4a359b79-e31e-488e-a272-3c8879736483"
       (reference "#PWR0117") (unit 1) (value "GND") (footprint "")
@@
       (reference "D3") (unit 1) (value "D_Schottky") (footprint "Diode_SMD:D_SOD-323")
     )
-    (path "/ced69235-8f7d-4667-bd55-c96b5907f8fa"
-      (reference "E1") (unit 1) (value "RotaryEncoder_Switch") (footprint "rotary_encoder")
-    )
     (path "/21946ec2-cae3-4116-acd9-40b9c5d1b38e"

Commit message: WIP
Connections:
- net -BATT is gone; now on net GND: J4.2 (Pin_2)
- net GND: no longer R7.2
- net VBUS: now also D2.2 (A)
- net CHRG_LED: no longer names the net of U3.1 (~{CHRG})
- net CHRG_LED: now also R7.2; no longer D2.2 (A)
Other:
- note removed: "Charging LED"
- moved on the sheet: D2, R7
Changed lines of the file:
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@@
   (junction (at 27.94 152.4) (diameter 0) (color 0 0 0 0)
+  )
+  (junction (at 245.11 24.13) (diameter 0) (color 0 0 0 0)
   )
   (junction (at 27.94 161.29) (diameter 0) (color 0 0 0 0)
@@
     (stroke (width 0) (type default) (color 0 0 0 0))
   )
-  (wire (pts (xy 241.3 36.83) (xy 245.11 36.83))
-    (stroke (width 0) (type default) (color 0 0 0 0))
-  )
   (wire (pts (xy 130.81 48.26) (xy 130.81 49.53))
     (stroke (width 0) (type default) (color 0 0 0 0))
@@
     (stroke (width 0) (type default) (color 0 0 0 0))
   )
+  (wire (pts (xy 240.03 36.83) (xy 245.11 36.83))
+    (stroke (width 0) (type default) (color 0 0 0 0))
+  )
   (wire (pts (xy 242.57 46.99) (xy 242.57 48.26))
     (stroke (width 0) (type default) (color 0 0 0 0))
   )
+  (wire (pts (xy 245.11 24.13) (xy 255.27 24.13))
+    (stroke (width 0) (type default) (color 0 0 0 0))
+  )
   (wire (pts (xy 27.94 175.26) (xy 27.94 171.45))
     (stroke (width 0) (type default) (color 0 0 0 0))
@@
     (stroke (width 0) (type default) (color 0 0 0 0))
   )
-  (wire (pts (xy 194.31 107.95) (xy 198.12 107.95))
+  (wire (pts (xy 234.95 31.75) (xy 234.95 36.83))
     (stroke (width 0) (type default) (color 0 0 0 0))
   )
@@
     (stroke (width 0) (type default) (color 0 0 0 0))
   )
-  (wire (pts (xy 255.27 26.67) (xy 255.27 29.21))
+  (wire (pts (xy 255.27 24.13) (xy 255.27 29.21))
     (stroke (width 0) (type default) (color 0 0 0 0))
   )
@@
   )
   (wire (pts (xy 124.46 147.32) (xy 124.46 146.05))
+    (stroke (width 0) (type default) (color 0 0 0 0))
+  )
+  (wire (pts (xy 234.95 24.13) (xy 245.11 24.13))
     (stroke (width 0) (type default) (color 0 0 0 0))
   )
@@
     (effects (font (size 2 2)) (justify left bottom))
   )
-  (text "Charging LED" (at 185.42 102.87 0)
-    (effects (font (size 1.7 1.7)) (justify left bottom))
-  )
   (text "Battery connector" (at 115.57 161.29 0)
     (effects (font (size 2 2)) (justify left bottom))
@@
     (effects (font (size 1.27 1.27)) (justify left bottom))
   )
-  (label "Net-(U3-PROG)" (at 242.57 41.91 90)
-    (effects (font (size 1.27 1.27)) (justify left bottom))
-  )
-  (label "Net-(D2-K)" (at 191.77 116.84 0)
-    (effects (font (size 1.27 1.27)) (justify left bottom))
+  (label "Net-(U3-PROG)" (at 242.57 40.64 180)
+    (effects (font (size 1.27 1.27)) (justify right bottom))
   )
   (label "unconnected-(U1-P0.19)" (at 55.88 99.06 270)
@@
     )
   )
-  (global_label "CHRG_LED" (shape input) (at 186.69 107.95 180) (fields_autoplaced)
-    (effects (font (size 1.27 1.27)) (justify right))
-    (property "Intersheet References" "${INTERSHEET_REFS}" (id 0) (at 174.8106 107.8706 0)
-      (effects (font (size 1.27 1.27)) (justify right) hide)
-    )
-  )
   (global_label "USBD+" (shape input) (at 135.89 48.26 0) (fields_autoplaced)
     (effects (font (size 1.27 1.27)) (justify left))
@@
     (effects (font (size 1.27 1.27)) (justify right))
     (property "Intersheet References" "${INTERSHEET_REFS}" (id 0) (at 28.1558 86.2806 0)
-      (effects (font (size 1.27 1.27)) (justify right) hide)
-    )
-  )
-  (global_label "CHRG_LED" (shape input) (at 241.3 36.83 180) (fields_autoplaced)
-    (effects (font (size 1.27 1.27)) (justify right))
-    (property "Intersheet References" "${INTERSHEET_REFS}" (id 0) (at 229.4206 36.7506 0)
       (effects (font (size 1.27 1.27)) (justify right) hide)
     )
@@
     (pin "1")
   )
-  (symbol (lib_id "power:GND") (at 203.2 107.95 90) (unit 1)
-    (in_bom yes) (on_board yes) (fields_autoplaced)
-    (property "Reference" "#PWR0130" (id 0) (at 209.55 107.95 0)
-      (effects (font (size 1.27 1.27)) hide)
-    )
-    (property "Value" "GND" (id 1) (at 207.01 107.9499 90)
-      (effects (font (size 1.27 1.27)) (justify right))
-    )
-    (property "Footprint" "" (id 2) (at 203.2 107.95 0)
-      (effects (font (size 1.27 1.27)) hide)
-    )
-    (property "Datasheet" "" (id 3) (at 203.2 107.95 0)
-      (effects (font (size 1.27 1.27)) hide)
-    )
-    (pin "1")
-  )
   (symbol (lib_id "Switch:SW_Push") (at 204.47 142.24 0) (unit 1)
     (in_bom yes) (on_board yes) (fields_autoplaced)
@@
     (pin "1")
   )
-  (symbol (lib_id "power:VBUS") (at 255.27 26.67 0) (unit 1)
-    (in_bom yes) (on_board yes) (fields_autoplaced)
-    (property "Reference" "#PWR0123" (id 0) (at 255.27 30.48 0)
-      (effects (font (size 1.27 1.27)) hide)
-    )
-    (property "Value" "VBUS" (id 1) (at 255.27 21.59 0))
-    (property "Footprint" "" (id 2) (at 255.27 26.67 0)
-      (effects (font (size 1.27 1.27)) hide)
-    )
-    (property "Datasheet" "" (id 3) (at 255.27 26.67 0)
+  (symbol (lib_id "power:VBUS") (at 245.11 24.13 0) (unit 1)
+    (in_bom yes) (on_board yes)
+    (property "Reference" "#PWR0123" (id 0) (at 245.11 27.94 0)
+      (effects (font (size 1.27 1.27)) hide)
+    )
+    (property "Value" "VBUS" (id 1) (at 245.11 20.32 0))
+    (property "Footprint" "" (id 2) (at 245.11 24.13 0)
+      (effects (font (size 1.27 1.27)) hide)
+    )
+    (property "Datasheet" "" (id 3) (at 245.11 24.13 0)
       (effects (font (size 1.27 1.27)) hide)
     )
@@
     (pin "1")
   )
-  (symbol (lib_id "power:-BATT") (at 125.73 167.64 90) (unit 1)
-    (in_bom yes) (on_board yes) (fields_autoplaced)
-    (property "Reference" "#PWR0113" (id 0) (at 129.54 167.64 0)
-      (effects (font (size 1.27 1.27)) hide)
-    )
-    (property "Value" "-BATT" (id 1) (at 121.92 167.6399 90)
-      (effects (font (size 1.27 1.27)) (justify left))
-    )
-    (property "Footprint" "" (id 2) (at 125.73 167.64 0)
-      (effects (font (size 1.27 1.27)) hide)
-    )
-    (property "Datasheet" "" (id 3) (at 125.73 167.64 0)
-      (effects (font (size 1.27 1.27)) hide)
-    )
-    (pin "1")
-  )
   (symbol (lib_id "Switch:SW_Push") (at 186.69 142.24 0) (unit 1)
     (in_bom yes) (on_board yes) (fields_autoplaced)
@@
     (pin "4")
   )
-  (symbol (lib_id "Device:LED") (at 190.5 107.95 180) (unit 1)
+  (symbol (lib_id "Device:LED") (at 234.95 27.94 90) (unit 1)
     (in_bom yes) (on_board yes)
-    (property "Reference" "D2" (id 0) (at 190.5 114.3 0))
-    (property "Value" "Red LED" (id 1) (at 190.5 111.76 0))
-    (property "Footprint" "LED_SMD:LED_0603_1608Metric" (id 2) (at 190.5 107.95 0)
-      (effects (font (size 1.27 1.27)) hide)
-    )
-    (property "Datasheet" "~" (id 3) (at 190.5 107.95 0)
+    (property "Reference" "D2" (id 0) (at 228.6 27.94 0))
+    (property "Value" "Red LED" (id 1) (at 231.14 27.94 0))
+    (property "Footprint" "LED_SMD:LED_0603_1608Metric" (id 2) (at 234.95 27.94 0)
+      (effects (font (size 1.27 1.27)) hide)
+    )
+    (property "Datasheet" "~" (id 3) (at 234.95 27.94 0)
       (effects (font (size 1.27 1.27)) hide)
     )
@@
     )
     (pin "1")
+    (pin "10")
     (pin "11")
     (pin "12")
@@
     (pin "7")
     (pin "8")
-    (pin "10")
     (pin "A1")
     (pin "A12")
@@
     (pin "S1")
   )
+  (symbol (lib_id "power:GND") (at 125.73 167.64 270) (unit 1)
+    (in_bom yes) (on_board yes)
+    (property "Reference" "#PWR?" (id 0) (at 119.38 167.64 0)
+      (effects (font (size 1.27 1.27)) hide)
+    )
+    (property "Value" "GND" (id 1) (at 118.11 167.64 90)
+      (effects (font (size 1.27 1.27)) (justify left))
+    )
+    (property "Footprint" "" (id 2) (at 125.73 167.64 0)
+      (effects (font (size 1.27 1.27)) hide)
+    )
+    (property "Datasheet" "" (id 3) (at 125.73 167.64 0)
+      (effects (font (size 1.27 1.27)) hide)
+    )
+    (pin "1")
+  )
   (symbol (lib_id "Switch:SW_Push") (at 270.51 176.53 0) (unit 1)
     (in_bom yes) (on_board yes) (fields_autoplaced)
@@
     (pin "2")
   )
-  (symbol (lib_id "Device:R_Small") (at 200.66 107.95 90) (unit 1)
+  (symbol (lib_id "Device:R_Small") (at 237.49 36.83 90) (unit 1)
     (in_bom yes) (on_board yes)
-    (property "Reference" "R7" (id 0) (at 205.74 105.41 90)
-      (effects (font (size 1.27 1.27)) (justify left))
-    )
-    (property "Value" "1K" (id 1) (at 201.93 105.41 90)
-      (effects (font (size 1.27 1.27)) (justify left))
-    )
-    (property "Footprint" "Resistor_SMD:R_0603_1608Metric" (id 2) (at 200.66 107.95 0)
-      (effects (font (size 1.27 1.27)) hide)
-    )
-    (property "Datasheet" "~" (id 3) (at 200.66 107.95 0)
+    (property "Reference" "R7" (id 0) (at 242.57 34.29 90)
+      (effects (font (size 1.27 1.27)) (justify left))
+    )
+    (property "Value" "1K" (id 1) (at 238.76 34.29 90)
+      (effects (font (size 1.27 1.27)) (justify left))
+    )
+    (property "Footprint" "Resistor_SMD:R_0603_1608Metric" (id 2) (at 237.49 36.83 0)
+      (effects (font (size 1.27 1.27)) hide)
+    )
+    (property "Datasheet" "~" (id 3) (at 237.49 36.83 0)
       (effects (font (size 1.27 1.27)) hide)
     )
@@
       (reference "#PWR0112") (unit 1) (value "+3.3V") (footprint "")
     )
-    (path "/a5a32878-9140-44a8-91cd-6dd680a16459"
-      (reference "#PWR0113") (unit 1) (value "-BATT") (footprint "")
-    )
     (path "/3cf0fbfd-66b2-4a7f-b06a-44415f8c69c1"
       (reference "#PWR0115") (unit 1) (value "GND") (footprint "")
@@
       (reference "#PWR0129") (unit 1) (value "GND") (footprint "")
     )
-    (path "/4ece50fa-7005-4669-adf7-9a16194f398a"
-      (reference "#PWR0130") (unit 1) (value "GND") (footprint "")
-    )
     (path "/5012d35e-3af9-4e53-b856-1b235e1f2af6"
       (reference "#PWR0131") (unit 1) (value "GND") (footprint "")
@@
       (reference "#PWR0145") (unit 1) (value "VBUS") (footprint "")
     )
+    (path "/c56b3a84-1bbd-4a7a-9aee-08c0176ce9bd"
+      (reference "#PWR?") (unit 1) (value "GND") (footprint "")
+    )
     (path "/73e1df8b-9e1b-43de-9821-06077b7495bd"

Commit message: WIP
Parts:
- added J5: USB, Connector_PinHeader_2.00mm:PinHeader_1x04_P2.00mm_Vertical, symbol Connector:Conn_01x04_Female
- SW1, SW10, SW11, SW12, SW13, SW14, SW15, SW16, SW17, SW2, SW3, SW4, SW5, SW6, SW7, SW8, SW9: footprint kicad-keyboard-parts:PG13500-reversible -> kiboard_cache:PG13500-reversible
Connections:
- net EXT_VCC: now also J5.1 (Pin_1)
- net GND: now also J5.2 (Pin_2)
- net P0.03: now reaches U1.6 (P0.03)
- net P0.03: now also J5.4 (Pin_4)
- net P0.02: now reaches U1.7 (P0.02)
- net P0.02: now also J5.3 (Pin_3)

Commit message: WIP
Connections:
- net SWDCLK: now also J2.3 (Pin_3); no longer J2.4 (Pin_4)
- net SWDIO: now also J2.4 (Pin_4); no longer J2.3 (Pin_3)
Changed lines of the file:
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@@
     )
   )
-  (global_label "SWDCLK" (shape input) (at 240.03 114.3 180) (fields_autoplaced)
-    (effects (font (size 1.27 1.27)) (justify right))
-    (property "Intersheet References" "${INTERSHEET_REFS}" (id 0) (at 230.2068 114.3794 0)
+  (global_label "SWDCLK" (shape input) (at 240.03 111.76 180) (fields_autoplaced)
+    (effects (font (size 1.27 1.27)) (justify right))
+    (property "Intersheet References" "${INTERSHEET_REFS}" (id 0) (at 230.2068 111.8394 0)
       (effects (font (size 1.27 1.27)) (justify right) hide)
     )
@@
     )
   )
-  (global_label "SWDIO" (shape input) (at 240.03 111.76 180) (fields_autoplaced)
-    (effects (font (size 1.27 1.27)) (justify right))
-    (property "Intersheet References" "${INTERSHEET_REFS}" (id 0) (at 231.8396 111.8394 0)
-      (effects (font (size 1.27 1.27)) (justify right) hide)
-    )
+  (global_label "SWDIO" (shape input) (at 240.03 114.3 180) (fields_autoplaced)
+    (effects (font (size 1.27 1.27)) (justify right))
+    (property "Intersheet References" "${INTERSHEET_REFS}" (id 0) (at 231.8396 114.3794 0)
+      (effects (font (size 1.27 1.27)) (justify right) hide)
+    )

Commit message: wip
Parts:
- added C3: 4.7n, Capacitor_SMD:C_1206_3216Metric, symbol Device:C_Small
- added R10: 1M, Resistor_SMD:R_0805_2012Metric, symbol Device:R_Small
- J1: value USB_C_Receptacle -> (none); footprint USB-C-12-Pin-MidMount -> (none); symbol Connector:USB_C_Receptacle -> Connector:USB_C_Receptacle_USB2.0
Connections:
- net Earth: now also C3.2, R10.2
- net GND: now also C3.1, R10.1; no longer J1.1 (GND), J1.12 (GND)
- net USBD+: now also J1.A6 (D+), J1.B6 (D+); no longer J1.6 (D+), J1.8 (D+)
- net USBD-: now also J1.A7 (D-), J1.B7 (D-); no longer J1.5 (D-), J1.7 (D-)
- net VBUS: now also J1.A4 (VBUS), J1.A9 (VBUS), J1.B4 (VBUS), J1.B9 (VBUS); no longer J1.11 (VBUS), J1.2 (VBUS)
- net Net-(J1-CC1): no longer names the net of R2.1
- net Net-(J1-CC1): now also J1.A5 (CC1); no longer J1.10 (CC1)
- net Net-(J1-CC2): no longer names the net of R1.1
- net Net-(J1-CC2): now also J1.B5 (CC2); no longer J1.4 (CC2)
- no-connect marks 11 -> 3
Other:
- note added: "Charging speed is affected by the value of R8"
- note removed: "Charging speed is affected by the value of R6"
- moved on the sheet: R1, R2
