File: KiCad/Bottom_Plate.kicad_pcb (KiCad board)
At the start: 2 copper layers, 140 x 91.2 mm, 9 parts

Commit message: wip
Parts:
- added ?: , clipboard:ade581d5-035f-4293-88b8-a7fbf49e45da, F.Cu at (179.4, 182.0)
- added ?: , clipboard:ade581d5-035f-4293-88b8-a7fbf49e45da, B.Cu at (155.1, 181.7)
Routing:
- added copper zone on B.Cu, net (none)
- added copper zone on F.Cu, net (none)
Other:
- board text added: "JLCJLCJLCJLC"

Commit message: wip
Parts:
- removed the ? at (179.4, 182.0)
- removed the ? at (155.1, 181.7)
- added ?: , clipboard:9b0fb884-d604-4a4e-b347-07e1aeb927c7, F.Cu at (174.2, 181.9)
- added ?: , clipboard:9b0fb884-d604-4a4e-b347-07e1aeb927c7, B.Cu at (160.5, 181.8)
